Commit message: full Quad + movement + launch

File: quadruped_description/urdf/bot_urdf_hii.xacro (robot description, xacro)
@@ -8,7 +8,7 @@
 <link name="base_link">
   <inertial>
-    <origin xyz="-0.23304185033712116 -0.030638440357548022 6.972053510835912e-05" rpy="0 0 0"/>
-    <mass value="3.992059884157941"/>
-    <inertia ixx="0.006111" iyy="0.083346" izz="0.084204" ixy="-0.000991" iyz="-3e-06" ixz="-7.3e-05"/>
+    <origin xyz="-0.006358858671583931 -0.003409645252810565 0.382156438627155" rpy="0 0 0"/>
+    <mass value="1.665624615569731"/>
+    <inertia ixx="0.010058" iyy="0.023588" izz="0.033004" ixy="0.0" iyz="0.0" ixz="0.000915"/>
   </inertial>
   <visual>
@@ -26,97 +26,245 @@
   </collision>
 </link>
-<link name="link2_v1_1">
-  <inertial>
-    <origin xyz="-0.07723046995547814 0.024997684987540944 3.1657101628697684e-08" rpy="0 0 0"/>
+<link name="lb1">
+  <inertial>
+    <origin xyz="-0.025499639213758474 -0.03608650849380332 0.008837273060876838" rpy="0 0 0"/>
+    <mass value="0.023765734421080365"/>
+    <inertia ixx="1.9e-05" iyy="1e-05" izz="2.1e-05" ixy="-0.0" iyz="4e-06" ixz="-0.0"/>
+  </inertial>
+  <visual>
+    <origin xyz="-0.159093 0.13841 -0.359825" rpy="0 0 0"/>
+    <geometry>
+      <mesh filename="file://$(find quadruped_description)/meshes/lb1_1.stl" scale="0.001 0.001 0.001"/>
+    </geometry>
+    <material name="silver"/>
+  </visual>
+  <collision>
+    <origin xyz="-0.159093 0.13841 -0.359825" rpy="0 0 0"/>
+    <geometry>
+      <mesh filename="file://$(find quadruped_description)/meshes/lb1_1.stl" scale="0.001 0.001 0.001"/>
+    </geometry>
+  </collision>
+</link>
+<link name="lf1">
+  <inertial>
+    <origin xyz="-0.025499639213758293 -0.03608650849380346 0.008837273060876838" rpy="0 0 0"/>
+    <mass value="0.023765734421080365"/>
+    <inertia ixx="1.9e-05" iyy="1e-05" izz="2.1e-05" ixy="-0.0" iyz="4e-06" ixz="-0.0"/>
+  </inertial>
+  <visual>
+    <origin xyz="0.085907 0.13841 -0.359825" rpy="0 0 0"/>
+    <geometry>
+      <mesh filename="file://$(find quadruped_description)/meshes/lf1_1.stl" scale="0.001 0.001 0.001"/>
+    </geometry>
+    <material name="silver"/>
+  </visual>
+  <collision>
+    <origin xyz="0.085907 0.13841 -0.359825" rpy="0 0 0"/>
+    <geometry>
+      <mesh filename="file://$(find quadruped_description)/meshes/lf1_1.stl" scale="0.001 0.001 0.001"/>
+    </geometry>
+  </collision>
+</link>
+<link name="rb1">
+  <inertial>
+    <origin xyz="-0.02549946018937349 0.03608721798818135 0.008837273060868067" rpy="0 0 0"/>
+    <mass value="0.023765734421080365"/>
+    <inertia ixx="1.9e-05" iyy="1e-05" izz="2.1e-05" ixy="-0.0" iyz="-4e-06" ixz="0.0"/>
+  </inertial>
+  <visual>
+    <origin xyz="-0.159093 -0.13159 -0.359825" rpy="0 0 0"/>
+    <geometry>
+      <mesh filename="file://$(find quadruped_description)/meshes/rb1_1.stl" scale="0.001 0.001 0.001"/>
+    </geometry>
+    <material name="silver"/>
+  </visual>
+  <collision>
+    <origin xyz="-0.159093 -0.13159 -0.359825" rpy="0 0 0"/>
+    <geometry>
+      <mesh filename="file://$(find quadruped_description)/meshes/rb1_1.stl" scale="0.001 0.001 0.001"/>
+    </geometry>
+  </collision>
+</link>
+<link name="rf1">
+  <inertial>
+    <origin xyz="-0.025499460189373144 0.0360872179881816 0.008837273060868123" rpy="0 0 0"/>
+    <mass value="0.023765734421080365"/>
+    <inertia ixx="1.9e-05" iyy="1e-05" izz="2.1e-05" ixy="-0.0" iyz="-4e-06" ixz="0.0"/>
+  </inertial>
+  <visual>
+    <origin xyz="0.085907 -0.13159 -0.359825" rpy="0 0 0"/>
+    <geometry>
+      <mesh filename="file://$(find quadruped_description)/meshes/rf1_1.stl" scale="0.001 0.001 0.001"/>
+    </geometry>
+    <material name="silver"/>
+  </visual>
+  <collision>
+    <origin xyz="0.085907 -0.13159 -0.359825" rpy="0 0 0"/>
+    <geometry>
+      <mesh filename="file://$(find quadruped_description)/meshes/rf1_1.stl" scale="0.001 0.001 0.001"/>
+    </geometry>
+  </collision>
+</link>
+<link name="lb2">
+  <inertial>
+    <origin xyz="4.4053550116163187e-07 -0.024997352134525086 -0.07676903071258923" rpy="0 0 0"/>
     <mass value="0.2750466774023333"/>
-    <inertia ixx="4.7e-05" iyy="0.000922" izz="0.00095" ixy="-0.0" iyz="-0.0" ixz="-0.0"/>
-  </inertial>
-  <visual>
-    <origin xyz="0.0 -0.082299 -0.001201" rpy="0 0 0"/>
-    <geometry>
-      <mesh filename="file://$(find quadruped_description)/meshes/link2_v1_1.stl" scale="0.001 0.001 0.001"/>
-    </geometry>
-    <material name="silver"/>
-  </visual>
-  <collision>
-    <origin xyz="0.0 -0.082299 -0.001201" rpy="0 0 0"/>
-    <geometry>
-      <mesh filename="file://$(find quadruped_description)/meshes/link2_v1_1.stl" scale="0.001 0.001 0.001"/>
-    </geometry>
-  </collision>
-</link>
-<link name="link3_1">
-  <inertial>
-    <origin xyz="-0.06999157163515277 0.02549464787405195 2.816749020764786e-07" rpy="0 0 0"/>
+    <inertia ixx="0.00095" iyy="0.000922" izz="4.7e-05" ixy="-0.0" iyz="-0.0" ixz="-0.0"/>
+  </inertial>
+  <visual>
+    <origin xyz="-0.133593 0.16741 -0.359825" rpy="0 0 0"/>
+    <geometry>
+      <mesh filename="file://$(find quadruped_description)/meshes/lb2_1.stl" scale="0.001 0.001 0.001"/>
+    </geometry>
+    <material name="silver"/>
+  </visual>
+  <collision>
+    <origin xyz="-0.133593 0.16741 -0.359825" rpy="0 0 0"/>
+    <geometry>
+      <mesh filename="file://$(find quadruped_description)/meshes/lb2_1.stl" scale="0.001 0.001 0.001"/>
+    </geometry>
+  </collision>
+</link>
+<link name="lf2">
+  <inertial>
+    <origin xyz="4.4053550139755426e-07 -0.02499735213452492 -0.076769030712589" rpy="0 0 0"/>
+    <mass value="0.2750466774023333"/>
+    <inertia ixx="0.00095" iyy="0.000922" izz="4.7e-05" ixy="-0.0" iyz="-0.0" ixz="-0.0"/>
+  </inertial>
+  <visual>
+    <origin xyz="0.111407 0.16741 -0.359825" rpy="0 0 0"/>
+    <geometry>
+      <mesh filename="file://$(find quadruped_description)/meshes/lf2_1.stl" scale="0.001 0.001 0.001"/>
+    </geometry>
+    <material name="silver"/>
+  </visual>
+  <collision>
+    <origin xyz="0.111407 0.16741 -0.359825" rpy="0 0 0"/>
+    <geometry>
+      <mesh filename="file://$(find quadruped_description)/meshes/lf2_1.stl" scale="0.001 0.001 0.001"/>
+    </geometry>
+  </collision>
+</link>
+<link name="rb2">
+  <inertial>
+    <origin xyz="4.405355014946988e-07 0.025002647865472988 -0.07676903071259905" rpy="0 0 0"/>
+    <mass value="0.2750466774023333"/>
+    <inertia ixx="0.00095" iyy="0.000922" izz="4.7e-05" ixy="-0.0" iyz="-0.0" ixz="-0.0"/>
+  </inertial>
+  <visual>
+    <origin xyz="-0.133593 -0.16059 -0.359825" rpy="0 0 0"/>
+    <geometry>
+      <mesh filename="file://$(find quadruped_description)/meshes/rb2_1.stl" scale="0.001 0.001 0.001"/>
+    </geometry>
+    <material name="silver"/>
+  </visual>
+  <collision>
+    <origin xyz="-0.133593 -0.16059 -0.359825" rpy="0 0 0"/>
+    <geometry>
+      <mesh filename="file://$(find quadruped_description)/meshes/rb2_1.stl" scale="0.001 0.001 0.001"/>
+    </geometry>
+  </collision>
+</link>
+<link name="rf2">
+  <inertial>
+    <origin xyz="4.4053550166123223e-07 0.025002647865473154 -0.07676903071259938" rpy="0 0 0"/>
+    <mass value="0.2750466774023333"/>
+    <inertia ixx="0.00095" iyy="0.000922" izz="4.7e-05" ixy="-0.0" iyz="-0.0" ixz="-0.0"/>
+  </inertial>
+  <visual>
+    <origin xyz="0.111407 -0.16059 -0.359825" rpy="0 0 0"/>
+    <geometry>
+      <mesh filename="file://$(find quadruped_description)/meshes/rf2_1.stl" scale="0.001 0.001 0.001"/>
+    </geometry>
+    <material name="silver"/>
+  </visual>
+  <collision>
+    <origin xyz="0.111407 -0.16059 -0.359825" rpy="0 0 0"/>
+    <geometry>
+      <mesh filename="file://$(find quadruped_description)/meshes/rf2_1.stl" scale="0.001 0.001 0.001"/>
+    </geometry>
+  </collision>
+</link>
+<link name="lb3">
+  <inertial>
+    <origin xyz="1.905177073602271e-07 -0.02550497548458827 -0.06999107230321813" rpy="0 0 0"/>
     <mass value="0.04435870319124352"/>
-    <inertia ixx="6e-06" iyy="6.3e-05" izz="6.5e-05" ixy="-0.0" iyz="0.0" ixz="-0.0"/>
-  </inertial>
-  <visual>
-    <origin xyz="0.154 -0.082299 -0.001201" rpy="0 0 0"/>
-    <geometry>
-      <mesh filename="file://$(find quadruped_description)/meshes/link3_1.stl" scale="0.001 0.001 0.001"/>
-    </geometry>
-    <material name="silver"/>
-  </visual>
-  <collision>
-    <origin xyz="0.154 -0.082299 -0.001201" rpy="0 0 0"/>
-    <geometry>
-      <mesh filename="file://$(find quadruped_description)/meshes/link3_1.stl" scale="0.001 0.001 0.001"/>
-    </geometry>
-  </collision>
-</link>
-<link name="link1_1">
-  <inertial>
-    <origin xyz="0.00883677372894309 0.036086841346824314 0.02549993238197565" rpy="0 0 0"/>
-    <mass value="0.023765734421080365"/>
-    <inertia ixx="2.1e-05" iyy="1e-05" izz="1.9e-05" ixy="-4e-06" iyz="0.0" ixz="-0.0"/>
-  </inertial>
-  <visual>
-    <origin xyz="0.0 -0.053299 0.024299" rpy="0 0 0"/>
-    <geometry>
-      <mesh filename="file://$(find quadruped_description)/meshes/link1_1.stl" scale="0.001 0.001 0.001"/>
-    </geometry>
-    <material name="silver"/>
-  </visual>
-  <collision>
-    <origin xyz="0.0 -0.053299 0.024299" rpy="0 0 0"/>
-    <geometry>
-      <mesh filename="file://$(find quadruped_description)/meshes/link1_1.stl" scale="0.001 0.001 0.001"/>
-    </geometry>
-  </collision>
-</link>
-<link name="leg_3_v1_1_fixed_ee"/>
-<!-- <link name="link1_rotated"/> -->
-<joint name="virtual_joint" type="fixed">
-  <origin xyz="0.0 0.0 1.0" rpy="0.0 -1.57 0.0"/>
-  <parent link="world"/>
-  <child link="base_link"/>
-</joint>
-<!-- <joint name="link1_rotated_joint" type="fixed">
-  <origin xyz="0.0 0.053299 -0.024299" rpy="0 0 3.14"/>
-  <parent link="base_link"/>
-  <child link="link1_rotated"/>
-</joint> -->
-<joint name="base_link1_joint" type="revolute">
-  <origin xyz="0.0 0.053299 -0.024299" rpy="0 0 0.0"/>
-  <parent link="base_link"/>
-  <child link="link1_1"/>
-  <axis xyz="0.0 0.0 1.0"/>
-  <limit upper="1.570796" lower="-1.570796" effort="100" velocity="100"/>
-</joint>
-<joint name="link1_link2_joint" type="revolute">
-  <origin xyz="0.0 0.029 0.0255" rpy="0 0 0"/>
-  <parent link="link1_1"/>
-  <child link="link2_v1_1"/>
-  <axis xyz="0.0 1.0 0.0"/>
-  <limit upper="1.570796" lower="-1.570796" effort="100" velocity="100"/>
-</joint>
-<joint name="link2_link3_joint" type="revolute">
-  <origin xyz="-0.154 0.0 0.0" rpy="0 0 0"/>
-  <parent link="link2_v1_1"/>
-  <child link="link3_1"/>
-  <axis xyz="0.0 1.0 0.0"/>
-  <limit upper="1.570796" lower="-1.570796" effort="100" velocity="100"/>
-</joint>
+    <inertia ixx="6.5e-05" iyy="6.3e-05" izz="6e-06" ixy="-0.0" iyz="-0.0" ixz="0.0"/>
+  </inertial>
+  <visual>
+    <origin xyz="-0.133593 0.16741 -0.205825" rpy="0 0 0"/>
+    <geometry>
+      <mesh filename="file://$(find quadruped_description)/meshes/lb3_1.stl" scale="0.001 0.001 0.001"/>
+    </geometry>
+    <material name="silver"/>
+  </visual>
+  <collision>
+    <origin xyz="-0.133593 0.16741 -0.205825" rpy="0 0 0"/>
+    <geometry>
+      <mesh filename="file://$(find quadruped_description)/meshes/lb3_1.stl" scale="0.001 0.001 0.001"/>
+    </geometry>
+  </collision>
+</link>
+<link name="lf3">
+  <inertial>
+    <origin xyz="1.905177022532012e-07 -0.025504975484588632 -0.06999107230321808" rpy="0 0 0"/>
+    <mass value="0.04435870319124352"/>
+    <inertia ixx="6.5e-05" iyy="6.3e-05" izz="6e-06" ixy="-0.0" iyz="-0.0" ixz="0.0"/>
+  </inertial>
+  <visual>
+    <origin xyz="0.111407 0.16741 -0.205825" rpy="0 0 0"/>
+    <geometry>
+      <mesh filename="file://$(find quadruped_description)/meshes/lf3_1.stl" scale="0.001 0.001 0.001"/>
+    </geometry>
+    <material name="silver"/>
+  </visual>
+  <collision>
+    <origin xyz="0.111407 0.16741 -0.205825" rpy="0 0 0"/>
+    <geometry>
+      <mesh filename="file://$(find quadruped_description)/meshes/lf3_1.stl" scale="0.001 0.001 0.001"/>
+    </geometry>
+  </collision>
+</link>
+<link name="rb3">
+  <inertial>
+    <origin xyz="7.100791705461074e-07 0.02550568497895228 -0.06999107230322818" rpy="0 0 0"/>
+    <mass value="0.04435870319124352"/>
+    <inertia ixx="6.5e-05" iyy="6.3e-05" izz="6e-06" ixy="-0.0" iyz="0.0" ixz="-0.0"/>
+  </inertial>
+  <visual>
+    <origin xyz="-0.133593 -0.16059 -0.205825" rpy="0 0 0"/>
+    <geometry>
+      <mesh filename="file://$(find quadruped_description)/meshes/rb3_1.stl" scale="0.001 0.001 0.001"/>
+    </geometry>
+    <material name="silver"/>
+  </visual>
+  <collision>
+    <origin xyz="-0.133593 -0.16059 -0.205825" rpy="0 0 0"/>
+    <geometry>
+      <mesh filename="file://$(find quadruped_description)/meshes/rb3_1.stl" scale="0.001 0.001 0.001"/>
+    </geometry>
+  </collision>
+</link>
+<link name="rf3">
+  <inertial>
+    <origin xyz="7.100791702685516e-07 0.025505684978952448 -0.06999107230322804" rpy="0 0 0"/>
+    <mass value="0.04435870319124352"/>
+    <inertia ixx="6.5e-05" iyy="6.3e-05" izz="6e-06" ixy="-0.0" iyz="0.0" ixz="-0.0"/>
+  </inertial>
+  <visual>
+    <origin xyz="0.111407 -0.16059 -0.205825" rpy="0 0 0"/>
+    <geometry>
+      <mesh filename="file://$(find quadruped_description)/meshes/rf3_1.stl" scale="0.001 0.001 0.001"/>
+    </geometry>
+    <material name="silver"/>
+  </visual>
+  <collision>
+    <origin xyz="0.111407 -0.16059 -0.205825" rpy="0 0 0"/>
+    <geometry>
+      <mesh filename="file://$(find quadruped_description)/meshes/rf3_1.stl" scale="0.001 0.001 0.001"/>
+    </geometry>
+  </collision>
+</link>
+<!-- <link name="leg_3_v1_1_fixed_ee"/> ise add krna hai for leg tip
 <joint name="Fixed_j" type="fixed">
   <origin xyz="-0.125 0.025 0.0" rpy="1.57 0 3.14"/>
@@ -124,4 +272,117 @@
   <child link="leg_3_v1_1_fixed_ee"/>
   <limit upper="1.570796" lower="-1.570796" effort="100" velocity="100"/>
+</joint> -->
+<joint name="virtual_joint" type="fixed">
+  <origin xyz="0.0 0.0 0.3" rpy="0.0 0.0 0.0"/>
+  <parent link="world"/>
+  <child link="base_link"/>
+</joint>
+<link name="leg_rb_tip"/>
+<link name="leg_rf_tip"/>
+<link name="leg_lb_tip"/>
+<link name="leg_lf_tip"/>
+<joint name="lb1_base" type="revolute">
+  <origin xyz="0.159093 -0.13841 0.359825" rpy="0 0 0"/>
+  <parent link="base_link"/>
+  <child link="lb1"/>
+  <axis xyz="1.0 0.0 0.0"/>
+  <limit upper="1.570796" lower="-1.570796" effort="100" velocity="100"/>
+</joint>
+<joint name="lf1_base" type="revolute">
+  <origin xyz="-0.085907 -0.13841 0.359825" rpy="0 0 0"/>
+  <parent link="base_link"/>
+  <child link="lf1"/>
+  <axis xyz="1.0 0.0 0.0"/>
+  <limit upper="1.570796" lower="-1.570796" effort="100" velocity="100"/>
+</joint>
+<joint name="rb1_base" type="revolute">
+  <origin xyz="0.159093 0.13159 0.359825" rpy="0 0 0"/>
+  <parent link="base_link"/>
+  <child link="rb1"/>
+  <axis xyz="-1.0 0.0 0.0"/>
+  <limit upper="1.570796" lower="-1.570796" effort="100" velocity="100"/>
+</joint>
+<joint name="rf1_base" type="revolute">
+  <origin xyz="-0.085907 0.13159 0.359825" rpy="0 0 0"/>
+  <parent link="base_link"/>
+  <child link="rf1"/>
+  <axis xyz="-1.0 0.0 0.0"/>
+  <limit upper="1.570796" lower="-1.570796" effort="100" velocity="100"/>
+</joint>
+<joint name="lb1_2" type="revolute">
+  <origin xyz="-0.0255 -0.029 0.0" rpy="0 0 0"/>
+  <parent link="lb1"/>
+  <child link="lb2"/>
+  <axis xyz="-0.0 -1.0 -0.0"/>
+  <limit upper="1.570796" lower="-1.570796" effort="100" velocity="100"/>
+</joint>
+<joint name="lf1_2" type="revolute">
+  <origin xyz="-0.0255 -0.029 0.0" rpy="0 0 0"/>
+  <parent link="lf1"/>
+  <child link="lf2"/>
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
File: quadruped_description/urdf/ros2_control.xacro (robot description, xacro)
@@ -5,5 +5,6 @@
             <plugin>gazebo_ros2_control/GazeboSystem</plugin>
         </hardware>
-        <joint name="base_link1_joint">
+        <!-- ******************************************* lb -->
+        <joint name="lb1_base">
             <command_interface name="position">
                 <param name="min">-1.57</param>
@@ -12,5 +13,5 @@
             <state_interface name="position"/>
         </joint>
-        <joint name="link1_link2_joint">
+        <joint name="lb1_2">
             <command_interface name="position">
                 <param name="min">-1.57</param>
@@ -19,5 +20,71 @@
             <state_interface name="position"/>
         </joint>
-        <joint name="link2_link3_joint">
+        <joint name="lb2_3">
+            <command_interface name="position">
+                <param name="min">-0.523</param>
+                <param name="max">2.61</param>
+            </command_interface>
+            <state_interface name="position"/>
+        </joint>
+        <!-- ******************************************* lf -->
+         <joint name="lf1_base">
+            <command_interface name="position">
+                <param name="min">-1.57</param>
+                <param name="max">1.57</param>
+            </command_interface>
+            <state_interface name="position"/>
+        </joint>
+        <joint name="lf1_2">
+            <command_interface name="position">
+                <param name="min">-1.57</param>
+                <param name="max">1.57</param>
+            </command_interface>
+            <state_interface name="position"/>
+        </joint>
+        <joint name="lf2_3">
+            <command_interface name="position">
+                <param name="min">-0.523</param>
+                <param name="max">2.61</param>
+            </command_interface>
+            <state_interface name="position"/>
+        </joint>
+        <!-- ******************************************* rb -->
+         <joint name="rb1_base">
+            <command_interface name="position">
+                <param name="min">-1.57</param>
+                <param name="max">1.57</param>
+            </command_interface>
+            <state_interface name="position"/>
+        </joint>
+        <joint name="rb1_2">
+            <command_interface name="position">
+                <param name="min">-1.57</param>
+                <param name="max">1.57</param>
+            </command_interface>
+            <state_interface name="position"/>
+        </joint>
+        <joint name="rb2_3">
+            <command_interface name="position">
+                <param name="min">-0.523</param>
+                <param name="max">2.61</param>
+            </command_interface>
+            <state_interface name="position"/>
+        </joint>
+        <!-- ******************************************* rf -->
+         <joint name="rf1_base">
+            <command_interface name="position">
+                <param name="min">-1.57</param>
+                <param name="max">1.57</param>
+            </command_interface>
+            <state_interface name="position"/>
+        </joint>
+        <joint name="rf1_2">
+            <command_interface name="position">
+                <param name="min">-1.57</param>
+                <param name="max">1.57</param>
+            </command_interface>
+            <state_interface name="position"/>
+        </joint>
+        <joint name="rf2_3">
             <command_interface name="position">
                 <param name="min">-0.523</param>
