Commit message: changed urdf files for gazebo

File: quadruped_description/urdf/bot_urdf_hii.xacro (robot description, xacro)
@@ -9,5 +9,5 @@
   <inertial>
     <origin xyz="-0.006358858671583931 -0.003409645252810565 0.382156438627155" rpy="0 0 0"/>
-    <mass value="1.665624615569731"/>
+    <mass value="1.6"/>
     <inertia ixx="0.010058" iyy="0.023588" izz="0.033004" ixy="0.0" iyz="0.0" ixz="0.000915"/>
   </inertial>
@@ -30,5 +30,6 @@
     <origin xyz="-0.025499639213758474 -0.03608650849380332 0.008837273060876838" rpy="0 0 0"/>
     <mass value="0.023765734421080365"/>
-    <inertia ixx="1.9e-05" iyy="1e-05" izz="2.1e-05" ixy="-0.0" iyz="4e-06" ixz="-0.0"/>
+    <!-- <inertia ixx="1.9e-05" iyy="1e-05" izz="2.1e-05" ixy="-0.0" iyz="4e-06" ixz="-0.0"/> -->
+        <inertia ixx="0.0" iyy="0.0" izz="0.0" ixy="-0.0" iyz="0.0" ixz="0.0"/>
   </inertial>
   <visual>
@@ -50,5 +51,6 @@
     <origin xyz="-0.025499639213758293 -0.03608650849380346 0.008837273060876838" rpy="0 0 0"/>
     <mass value="0.023765734421080365"/>
-    <inertia ixx="1.9e-05" iyy="1e-05" izz="2.1e-05" ixy="-0.0" iyz="4e-06" ixz="-0.0"/>
+    <!-- <inertia ixx="1.9e-05" iyy="1e-05" izz="2.1e-05" ixy="-0.0" iyz="4e-06" ixz="-0.0"/> -->
+        <inertia ixx="0.0" iyy="0.0" izz="0.0" ixy="-0.0" iyz="0.0" ixz="0.0"/>
   </inertial>
   <visual>
@@ -70,5 +72,6 @@
     <origin xyz="-0.02549946018937349 0.03608721798818135 0.008837273060868067" rpy="0 0 0"/>
     <mass value="0.023765734421080365"/>
-    <inertia ixx="1.9e-05" iyy="1e-05" izz="2.1e-05" ixy="-0.0" iyz="-4e-06" ixz="0.0"/>
+    <!-- <inertia ixx="1.9e-05" iyy="1e-05" izz="2.1e-05" ixy="-0.0" iyz="-4e-06" ixz="0.0"/> -->
+        <inertia ixx="0.0" iyy="0.0" izz="0.0" ixy="-0.0" iyz="0.0" ixz="0.0"/>
   </inertial>
   <visual>
@@ -90,5 +93,6 @@
     <origin xyz="-0.025499460189373144 0.0360872179881816 0.008837273060868123" rpy="0 0 0"/>
     <mass value="0.023765734421080365"/>
-    <inertia ixx="1.9e-05" iyy="1e-05" izz="2.1e-05" ixy="-0.0" iyz="-4e-06" ixz="0.0"/>
+    <!-- <inertia ixx="1.9e-05" iyy="1e-05" izz="2.1e-05" ixy="-0.0" iyz="-4e-06" ixz="0.0"/> -->
+    <inertia ixx="0.0" iyy="0.0" izz="0.0" ixy="-0.0" iyz="0.0" ixz="0.0"/>
   </inertial>
   <visual>
@@ -278,8 +282,100 @@
   <child link="base_link"/>
 </joint>
-<link name="leg_rb_tip"/>
-<link name="leg_rf_tip"/>
-<link name="leg_lb_tip"/>
-<link name="leg_lf_tip"/>
+<link name="leg_rb_tip">
+<!-- <visual>
+            <origin rpy="0 0 0" xyz="0 0 0"/>
+            <geometry>
+                <sphere radius="0.016"/>
+            </geometry>
+            <material name="orange"/>
+        </visual>
+        <collision>
+            <origin rpy="0 0 0" xyz="0 0 0"/>
+            <geometry>
+                <sphere radius="0.016"/>
+            </geometry>
+            <surface>
+                <friction>
+                    <ode>
+                        <mu>100</mu>
+                        <mu2>100</mu2>
+                        <fdir1>1 0 0</fdir1>
+                    </ode>
+                </friction>
+            </surface>
+        </collision> -->
+</link>
+<link name="leg_rf_tip">
+<!-- <visual>
+            <origin rpy="0 0 0" xyz="0 0 0"/>
+            <geometry>
+                <sphere radius="0.016"/>
+            </geometry>
+            <material name="orange"/>
+        </visual>
+        <collision>
+            <origin rpy="0 0 0" xyz="0 0 0"/>
+            <geometry>
+                <sphere radius="0.016"/>
+            </geometry>
+            <surface>
+                <friction>
+                    <ode>
+                        <mu>100</mu>
+                        <mu2>100</mu2>
+                        <fdir1>1 0 0</fdir1>
+                    </ode>
+                </friction>
+            </surface>
+        </collision> -->
+</link>
+<link name="leg_lb_tip">
+<!-- <visual>
+            <origin rpy="0 0 0" xyz="0 0 0"/>
+            <geometry>
+                <sphere radius="0.016"/>
+            </geometry>
+            <material name="orange"/>
+        </visual>
+        <collision>
+            <origin rpy="0 0 0" xyz="0 0 0"/>
+            <geometry>
+                <sphere radius="0.016"/>
+            </geometry>
+            <surface>
+                <friction>
+                    <ode>
+                        <mu>100</mu>
+                        <mu2>100</mu2>
+                        <fdir1>1 0 0</fdir1>
+                    </ode>
+                </friction>
+            </surface>
+        </collision> -->
+</link>
+<link name="leg_lf_tip">
+<!-- <visual>
+            <origin rpy="0 0 0" xyz="0 0 0"/>
+            <geometry>
+                <sphere radius="0.016"/>
+            </geometry>
+            <material name="orange"/>
+        </visual>
+        <collision>
+            <origin rpy="0 0 0" xyz="0 0 0"/>
+            <geometry>
+                <sphere radius="0.016"/>
+            </geometry>
+            <surface>
+                <friction>
+                    <ode>
+                        <mu>100</mu>
+                        <mu2>100</mu2>
+                        <fdir1>1 0 0</fdir1>
+                    </ode>
+                </friction>
+            </surface>
+        </collision> -->
+</link>
 <joint name="lb1_base" type="revolute">
   <origin xyz="0.159093 -0.13841 0.359825" rpy="0 0 0"/>

Commit message: hardware

File: quadruped_description/urdf/bot_urdf_hii.xacro (robot description, xacro)
@@ -1,15 +1,26 @@
 <?xml version="1.0" ?>
 <robot name="FusionComponent" xmlns:xacro="http://www.ros.org/wiki/xacro">
+<xacro:arg name="is_sim" default="false"/>
 <xacro:include filename="$(find quadruped_description)/urdf/materials.xacro" />
 <!-- <xacro:include filename="$(find quadruped_description)/urdf/bot_urdf_hii.trans" /> -->
 <xacro:include filename="$(find quadruped_description)/urdf/bot_urdf_hii.gazebo" />
 <xacro:include filename="$(find quadruped_description)/urdf/ros2_control.xacro" />
-<link name="world"></link>
+<xacro:macro name="box_inertia" params="m l w h xyz rpy">
+  <inertial>
+    <origin xyz="${xyz}" rpy="${rpy}" />
+    <mass value="${m}" />
+    <inertia ixx="${(m/12)*(h*h + l*l)}" ixy="0" ixz="0"
+              iyy="${(m/12)*(w*w +l*l)}" iyz="0"
+              izz="${(m/12)*(w*w + h*h)}" />
+  </inertial>
+</xacro:macro>
+<!-- <link name="world"></link> -->
 <link name="base_link">
-  <inertial>
-    <origin xyz="-0.006358858671583931 -0.003409645252810565 0.382156438627155" rpy="0 0 0"/>
-    <mass value="1.6"/>
-    <inertia ixx="0.010058" iyy="0.023588" izz="0.033004" ixy="0.0" iyz="0.0" ixz="0.000915"/>
-  </inertial>
+  <!-- <inertial>
+    <origin xyz="0.01 0.0 0.3459" rpy="0 0 0"/>
+    <mass value="2.5"/>
+    <inertia ixx="0.02245" iyy="0.02245" izz="0.02245" ixy="0.0" iyz="0.0" ixz="0.0"/>
+  </inertial> -->
+  <xacro:box_inertia m="1.0" l="0.10" w="0.244" h="0.27" xyz="0.01 0.0 0.3459" rpy="0 0 0" />
   <visual>
     <origin xyz="0 0 0" rpy="0 0 0"/>
@@ -29,7 +40,7 @@
   <inertial>
     <origin xyz="-0.025499639213758474 -0.03608650849380332 0.008837273060876838" rpy="0 0 0"/>
-    <mass value="0.023765734421080365"/>
-    <!-- <inertia ixx="1.9e-05" iyy="1e-05" izz="2.1e-05" ixy="-0.0" iyz="4e-06" ixz="-0.0"/> -->
-        <inertia ixx="0.0" iyy="0.0" izz="0.0" ixy="-0.0" iyz="0.0" ixz="0.0"/>
+    <mass value="0.01"/>
+    <!-- <inertia ixx="1.9e-05" iyy="1.9e-05" izz="1.9e-05" ixy="0.0" iyz="0.0" ixz="0.0"/> -->
+    <inertia ixx="0.0" iyy="0.0" izz="0.0" ixy="0.0" iyz="0.0" ixz="0.0"/>
   </inertial>
   <visual>
@@ -50,7 +61,7 @@
   <inertial>
     <origin xyz="-0.025499639213758293 -0.03608650849380346 0.008837273060876838" rpy="0 0 0"/>
-    <mass value="0.023765734421080365"/>
-    <!-- <inertia ixx="1.9e-05" iyy="1e-05" izz="2.1e-05" ixy="-0.0" iyz="4e-06" ixz="-0.0"/> -->
-        <inertia ixx="0.0" iyy="0.0" izz="0.0" ixy="-0.0" iyz="0.0" ixz="0.0"/>
+    <mass value="0.01"/>
+    <!-- <inertia ixx="1.9e-05" iyy="1.9e-05" izz="1.9e-05" ixy="0.0" iyz="0.0" ixz="0.0"/> -->
+    <inertia ixx="0.0" iyy="0.0" izz="0.0" ixy="0.0" iyz="0.0" ixz="0.0"/>
   </inertial>
   <visual>
@@ -71,7 +82,7 @@
   <inertial>
     <origin xyz="-0.02549946018937349 0.03608721798818135 0.008837273060868067" rpy="0 0 0"/>
-    <mass value="0.023765734421080365"/>
-    <!-- <inertia ixx="1.9e-05" iyy="1e-05" izz="2.1e-05" ixy="-0.0" iyz="-4e-06" ixz="0.0"/> -->
-        <inertia ixx="0.0" iyy="0.0" izz="0.0" ixy="-0.0" iyz="0.0" ixz="0.0"/>
+    <mass value="0.01"/>
+    <!-- <inertia ixx="1.9e-05" iyy="1.9e-05" izz="1.9e-05" ixy="0.0" iyz="0.0" ixz="0.0"/> -->
+    <inertia ixx="0.0" iyy="0.0" izz="0.0" ixy="0.0" iyz="0.0" ixz="0.0"/>
   </inertial>
   <visual>
@@ -92,7 +103,7 @@
   <inertial>
     <origin xyz="-0.025499460189373144 0.0360872179881816 0.008837273060868123" rpy="0 0 0"/>
-    <mass value="0.023765734421080365"/>
-    <!-- <inertia ixx="1.9e-05" iyy="1e-05" izz="2.1e-05" ixy="-0.0" iyz="-4e-06" ixz="0.0"/> -->
-    <inertia ixx="0.0" iyy="0.0" izz="0.0" ixy="-0.0" iyz="0.0" ixz="0.0"/>
+    <mass value="0.01"/>
+    <!-- <inertia ixx="1.9e-05" iyy="1.9e-05" izz="1.9e-05" ixy="0.0" iyz="0.0" ixz="0.0"/> -->
+    <inertia ixx="0.0" iyy="0.0" izz="0.0" ixy="0.0" iyz="0.0" ixz="0.0"/>
   </inertial>
   <visual>
@@ -112,7 +123,8 @@
 <link name="lb2">
   <inertial>
-    <origin xyz="4.4053550116163187e-07 -0.024997352134525086 -0.07676903071258923" rpy="0 0 0"/>
-    <mass value="0.2750466774023333"/>
-    <inertia ixx="0.00095" iyy="0.000922" izz="4.7e-05" ixy="-0.0" iyz="-0.0" ixz="-0.0"/>
+    <origin xyz="4.4053550116163187e-07 -0.024997352134525086 -0.058" rpy="0 0 0"/>
+    <mass value="0.1"/>
+    <!-- <inertia ixx="0.00095" iyy="0.000922" izz="4.7e-05" ixy="-0.0" iyz="-0.0" ixz="-0.0"/> -->
+    <inertia ixx="0.0" iyy="0.0" izz="0.0" ixy="0.0" iyz="0.0" ixz="0.0"/>
   </inertial>
   <visual>
@@ -132,7 +144,8 @@
 <link name="lf2">
   <inertial>
-    <origin xyz="4.4053550139755426e-07 -0.02499735213452492 -0.076769030712589" rpy="0 0 0"/>
-    <mass value="0.2750466774023333"/>
-    <inertia ixx="0.00095" iyy="0.000922" izz="4.7e-05" ixy="-0.0" iyz="-0.0" ixz="-0.0"/>
+    <origin xyz="4.4053550139755426e-07 -0.02499735213452492 -0.058" rpy="0 0 0"/>
+    <mass value="0.1"/>
+    <!-- <inertia ixx="0.00095" iyy="0.000922" izz="4.7e-05" ixy="-0.0" iyz="-0.0" ixz="-0.0"/> -->
+    <inertia ixx="0.0" iyy="0.0" izz="0.0" ixy="0.0" iyz="0.0" ixz="0.0"/>
   </inertial>
   <visual>
@@ -152,7 +165,8 @@
 <link name="rb2">
   <inertial>
-    <origin xyz="4.405355014946988e-07 0.025002647865472988 -0.07676903071259905" rpy="0 0 0"/>
-    <mass value="0.2750466774023333"/>
-    <inertia ixx="0.00095" iyy="0.000922" izz="4.7e-05" ixy="-0.0" iyz="-0.0" ixz="-0.0"/>
+    <origin xyz="4.405355014946988e-07 0.025002647865472988 -0.058" rpy="0 0 0"/>
+    <mass value="0.1"/>
+    <!-- <inertia ixx="0.00095" iyy="0.000922" izz="4.7e-05" ixy="-0.0" iyz="-0.0" ixz="-0.0"/> -->
+    <inertia ixx="0.0" iyy="0.0" izz="0.0" ixy="0.0" iyz="0.0" ixz="0.0"/>
   </inertial>
   <visual>
@@ -171,9 +185,11 @@
 </link>
 <link name="rf2">
-  <inertial>
-    <origin xyz="4.4053550166123223e-07 0.025002647865473154 -0.07676903071259938" rpy="0 0 0"/>
-    <mass value="0.2750466774023333"/>
-    <inertia ixx="0.00095" iyy="0.000922" izz="4.7e-05" ixy="-0.0" iyz="-0.0" ixz="-0.0"/>
-  </inertial>
+  <!-- <inertial>
+    <origin xyz="4.4053550166123223e-07 0.025002647865473154 -0.058" rpy="0 0 0"/>
+    <mass value="0.1"/> -->
+    <!-- <inertia ixx="0.00095" iyy="0.000922" izz="4.7e-05" ixy="-0.0" iyz="-0.0" ixz="-0.0"/> -->
+    <!-- <inertia ixx="0.0" iyy="0.0" izz="0.0" ixy="0.0" iyz="0.0" ixz="0.0"/>
+  </inertial> -->
+  <xacro:box_inertia m="0.1" l="0.10" w="0.03" h="0.03" xyz="1.905177073602271e-07 -0.02550497548458827 -0.06999107230321813" rpy="0 0 0" />
   <visual>
     <origin xyz="0.111407 -0.16059 -0.359825" rpy="0 0 0"/>
@@ -191,9 +207,11 @@
 </link>
 <link name="lb3">
-  <inertial>
+  <!-- <inertial>
     <origin xyz="1.905177073602271e-07 -0.02550497548458827 -0.06999107230321813" rpy="0 0 0"/>
-    <mass value="0.04435870319124352"/>
-    <inertia ixx="6.5e-05" iyy="6.3e-05" izz="6e-06" ixy="-0.0" iyz="-0.0" ixz="0.0"/>
-  </inertial>
+    <mass value="0.1"/>
+    <inertia ixx="6.5e-05" iyy="6.3e-05" izz="6e-06" ixy="-0.0" iyz="-0.0" ixz="0.0"/> -->
+    <!-- <inertia ixx="0.0" iyy="0.0" izz="0.0" ixy="0.0" iyz="0.0" ixz="0.0"/> -->
+  <!-- </inertial> -->
+  <xacro:box_inertia m="0.1" l="0.10" w="0.03" h="0.03" xyz="1.905177073602271e-07 -0.02550497548458827 -0.06999107230321813" rpy="0 0 0" />
   <visual>
     <origin xyz="-0.133593 0.16741 -0.205825" rpy="0 0 0"/>
@@ -211,9 +229,11 @@
 </link>
 <link name="lf3">
-  <inertial>
+  <!-- <inertial>
     <origin xyz="1.905177022532012e-07 -0.025504975484588632 -0.06999107230321808" rpy="0 0 0"/>
-    <mass value="0.04435870319124352"/>
-    <inertia ixx="6.5e-05" iyy="6.3e-05" izz="6e-06" ixy="-0.0" iyz="-0.0" ixz="0.0"/>
-  </inertial>
+    <mass value="0.1"/>
+    <inertia ixx="6.5e-05" iyy="6.3e-05" izz="6e-06" ixy="-0.0" iyz="-0.0" ixz="0.0"/> -->
+    <!-- <inertia ixx="0.0" iyy="0.0" izz="0.0" ixy="0.0" iyz="0.0" ixz="0.0"/> -->
+  <!-- </inertial> -->
+  <xacro:box_inertia m="0.1" l="0.10" w="0.03" h="0.03" xyz="1.905177022532012e-07 -0.025504975484588632 -0.06999107230321808" rpy="0 0 0" />
   <visual>
     <origin xyz="0.111407 0.16741 -0.205825" rpy="0 0 0"/>
@@ -231,9 +251,11 @@
 </link>
 <link name="rb3">
-  <inertial>
+  <!-- <inertial>
     <origin xyz="7.100791705461074e-07 0.02550568497895228 -0.06999107230322818" rpy="0 0 0"/>
-    <mass value="0.04435870319124352"/>
-    <inertia ixx="6.5e-05" iyy="6.3e-05" izz="6e-06" ixy="-0.0" iyz="0.0" ixz="-0.0"/>
-  </inertial>
+    <mass value="0.1"/>
+    <inertia ixx="6.5e-05" iyy="6.3e-05" izz="6e-06" ixy="-0.0" iyz="0.0" ixz="-0.0"/> -->
+    <!-- <inertia ixx="0.0" iyy="0.0" izz="0.0" ixy="0.0" iyz="0.0" ixz="0.0"/> -->
+  <!-- </inertial> -->
+  <xacro:box_inertia m="0.1" l="0.10" w="0.03" h="0.03" xyz="7.100791705461074e-07 0.02550568497895228 -0.06999107230322818" rpy="0 0 0" />
   <visual>
     <origin xyz="-0.133593 -0.16059 -0.205825" rpy="0 0 0"/>
@@ -251,9 +273,11 @@
 </link>
 <link name="rf3">
-  <inertial>
+  <!-- <inertial>
     <origin xyz="7.100791702685516e-07 0.025505684978952448 -0.06999107230322804" rpy="0 0 0"/>
-    <mass value="0.04435870319124352"/>
-    <inertia ixx="6.5e-05" iyy="6.3e-05" izz="6e-06" ixy="-0.0" iyz="0.0" ixz="-0.0"/>
-  </inertial>
+    <mass value="0.1"/>
+    <inertia ixx="6.5e-05" iyy="6.3e-05" izz="6e-06" ixy="-0.0" iyz="0.0" ixz="-0.0"/> -->
+    <!-- <inertia ixx="0.0" iyy="0.0" izz="0.0" ixy="0.0" iyz="0.0" ixz="0.0"/> -->
+  <!-- </inertial> -->
+  <xacro:box_inertia m="0.1" l="0.10" w="0.03" h="0.03" xyz="7.100791702685516e-07 0.025505684978952448 -0.06999107230322804" rpy="0 0 0" />
   <visual>
     <origin xyz="0.111407 -0.16059 -0.205825" rpy="0 0 0"/>
@@ -277,11 +301,11 @@
   <limit upper="1.570796" lower="-1.570796" effort="100" velocity="100"/>
 </joint> -->
-<joint name="virtual_joint" type="fixed">
+<!-- <joint name="virtual_joint" type="fixed">
   <origin xyz="0.0 0.0 0.3" rpy="0.0 0.0 0.0"/>
   <parent link="world"/>
   <child link="base_link"/>
-</joint>
+</joint> -->
 <link name="leg_rb_tip">
-<!-- <visual>
+<visual>
             <origin rpy="0 0 0" xyz="0 0 0"/>
             <geometry>
@@ -298,14 +322,14 @@
                 <friction>
                     <ode>
-                        <mu>100</mu>
-                        <mu2>100</mu2>
+                        <mu>0.6</mu>
+                        <mu2>0.6</mu2>
                         <fdir1>1 0 0</fdir1>
                     </ode>
                 </friction>
             </surface>
-        </collision> -->
+        </collision>
 </link>
 <link name="leg_rf_tip">
-<!-- <visual>
+<visual>
             <origin rpy="0 0 0" xyz="0 0 0"/>
             <geometry>
@@ -322,14 +346,14 @@
                 <friction>
                     <ode>
-                        <mu>100</mu>
-                        <mu2>100</mu2>
+                        <mu>0.6</mu>
+                        <mu2>0.6</mu2>
                         <fdir1>1 0 0</fdir1>
                     </ode>
                 </friction>
             </surface>
-        </collision> -->
+        </collision>
 </link>
 <link name="leg_lb_tip">
-<!-- <visual>
+<visual>
             <origin rpy="0 0 0" xyz="0 0 0"/>
             <geometry>
@@ -346,14 +370,14 @@
                 <friction>
                     <ode>
-                        <mu>100</mu>
-                        <mu2>100</mu2>
+                        <mu>0.6</mu>
+                        <mu2>0.6</mu2>
                         <fdir1>1 0 0</fdir1>
                     </ode>
                 </friction>
             </surface>
-        </collision> -->
+        </collision>
 </link>
 <link name="leg_lf_tip">
-<!-- <visual>
+<visual>
             <origin rpy="0 0 0" xyz="0 0 0"/>
             <geometry>
@@ -370,11 +394,11 @@
                 <friction>
                     <ode>
-                        <mu>100</mu>
-                        <mu2>100</mu2>
+                        <mu>0.6</mu>
+                        <mu2>0.6</mu2>
                         <fdir1>1 0 0</fdir1>
                     </ode>
                 </friction>
             </surface>
-        </collision> -->
+        </collision>
 </link>
 <joint name="lb1_base" type="revolute">

File: quadruped_description/urdf/ros2_control.xacro (robot description, xacro)
@@ -2,7 +2,15 @@
 <robot xmlns:xacro="http://www.ros.org/wiki/xacro">
     <ros2_control name="GazeboSystem" type="system">
-        <hardware>
-            <plugin>gazebo_ros2_control/GazeboSystem</plugin>
-        </hardware>
+        <xacro:if value="$(eval is_sim)">
+            <hardware>
+                <plugin>gazebo_ros2_control/GazeboSystem</plugin>
+            </hardware>
+        </xacro:if>
+        <xacro:if value="$(eval not is_sim)">
+            <hardware>
+                <plugin>bumperbot_controller/RobotInterface</plugin>
+                <param name="port">/dev/ttyACM0</param>
+            </hardware>
+        </xacro:if>
         <!-- ******************************************* lb -->
         <joint name="lb1_base">

Commit message: added odometry logic

File: quadruped_description/urdf/bot_urdf_hii.xacro (robot description, xacro)
@@ -1,5 +1,5 @@
 <?xml version="1.0" ?>
 <robot name="FusionComponent" xmlns:xacro="http://www.ros.org/wiki/xacro">
-<xacro:arg name="is_sim" default="false"/>
+<xacro:arg name="is_sim" default="true"/>
 <xacro:include filename="$(find quadruped_description)/urdf/materials.xacro" />
 <!-- <xacro:include filename="$(find quadruped_description)/urdf/bot_urdf_hii.trans" /> -->
@@ -15,5 +15,5 @@
   </inertial>
 </xacro:macro>
-<!-- <link name="world"></link> -->
+<link name="world"></link>
 <link name="base_link">
   <!-- <inertial>
@@ -41,6 +41,6 @@
     <origin xyz="-0.025499639213758474 -0.03608650849380332 0.008837273060876838" rpy="0 0 0"/>
     <mass value="0.01"/>
-    <!-- <inertia ixx="1.9e-05" iyy="1.9e-05" izz="1.9e-05" ixy="0.0" iyz="0.0" ixz="0.0"/> -->
-    <inertia ixx="0.0" iyy="0.0" izz="0.0" ixy="0.0" iyz="0.0" ixz="0.0"/>
+    <inertia ixx="1.9e-05" iyy="1.9e-05" izz="1.9e-05" ixy="0.0" iyz="0.0" ixz="0.0"/>
+    <!-- <inertia ixx="0.0" iyy="0.0" izz="0.0" ixy="0.0" iyz="0.0" ixz="0.0"/> -->
   </inertial>
   <visual>
@@ -62,6 +62,6 @@
     <origin xyz="-0.025499639213758293 -0.03608650849380346 0.008837273060876838" rpy="0 0 0"/>
     <mass value="0.01"/>
-    <!-- <inertia ixx="1.9e-05" iyy="1.9e-05" izz="1.9e-05" ixy="0.0" iyz="0.0" ixz="0.0"/> -->
-    <inertia ixx="0.0" iyy="0.0" izz="0.0" ixy="0.0" iyz="0.0" ixz="0.0"/>
+    <inertia ixx="1.9e-05" iyy="1.9e-05" izz="1.9e-05" ixy="0.0" iyz="0.0" ixz="0.0"/>
+    <!-- <inertia ixx="0.0" iyy="0.0" izz="0.0" ixy="0.0" iyz="0.0" ixz="0.0"/> -->
   </inertial>
   <visual>
@@ -83,6 +83,6 @@
     <origin xyz="-0.02549946018937349 0.03608721798818135 0.008837273060868067" rpy="0 0 0"/>
     <mass value="0.01"/>
-    <!-- <inertia ixx="1.9e-05" iyy="1.9e-05" izz="1.9e-05" ixy="0.0" iyz="0.0" ixz="0.0"/> -->
-    <inertia ixx="0.0" iyy="0.0" izz="0.0" ixy="0.0" iyz="0.0" ixz="0.0"/>
+    <inertia ixx="1.9e-05" iyy="1.9e-05" izz="1.9e-05" ixy="0.0" iyz="0.0" ixz="0.0"/>
+    <!-- <inertia ixx="0.0" iyy="0.0" izz="0.0" ixy="0.0" iyz="0.0" ixz="0.0"/> -->
   </inertial>
   <visual>
@@ -104,6 +104,6 @@
     <origin xyz="-0.025499460189373144 0.0360872179881816 0.008837273060868123" rpy="0 0 0"/>
     <mass value="0.01"/>
-    <!-- <inertia ixx="1.9e-05" iyy="1.9e-05" izz="1.9e-05" ixy="0.0" iyz="0.0" ixz="0.0"/> -->
-    <inertia ixx="0.0" iyy="0.0" izz="0.0" ixy="0.0" iyz="0.0" ixz="0.0"/>
+    <inertia ixx="1.9e-05" iyy="1.9e-05" izz="1.9e-05" ixy="0.0" iyz="0.0" ixz="0.0"/>
+    <!-- <inertia ixx="0.0" iyy="0.0" izz="0.0" ixy="0.0" iyz="0.0" ixz="0.0"/> -->
   </inertial>
   <visual>
@@ -125,6 +125,6 @@
     <origin xyz="4.4053550116163187e-07 -0.024997352134525086 -0.058" rpy="0 0 0"/>
     <mass value="0.1"/>
-    <!-- <inertia ixx="0.00095" iyy="0.000922" izz="4.7e-05" ixy="-0.0" iyz="-0.0" ixz="-0.0"/> -->
-    <inertia ixx="0.0" iyy="0.0" izz="0.0" ixy="0.0" iyz="0.0" ixz="0.0"/>
+    <inertia ixx="0.00095" iyy="0.000922" izz="4.7e-05" ixy="-0.0" iyz="-0.0" ixz="-0.0"/>
+    <!-- <inertia ixx="0.0" iyy="0.0" izz="0.0" ixy="0.0" iyz="0.0" ixz="0.0"/> -->
   </inertial>
   <visual>
@@ -146,6 +146,6 @@
     <origin xyz="4.4053550139755426e-07 -0.02499735213452492 -0.058" rpy="0 0 0"/>
     <mass value="0.1"/>
-    <!-- <inertia ixx="0.00095" iyy="0.000922" izz="4.7e-05" ixy="-0.0" iyz="-0.0" ixz="-0.0"/> -->
-    <inertia ixx="0.0" iyy="0.0" izz="0.0" ixy="0.0" iyz="0.0" ixz="0.0"/>
+    <inertia ixx="0.00095" iyy="0.000922" izz="4.7e-05" ixy="-0.0" iyz="-0.0" ixz="-0.0"/>
+    <!-- <inertia ixx="0.0" iyy="0.0" izz="0.0" ixy="0.0" iyz="0.0" ixz="0.0"/> -->
   </inertial>
   <visual>
@@ -167,6 +167,6 @@
     <origin xyz="4.405355014946988e-07 0.025002647865472988 -0.058" rpy="0 0 0"/>
     <mass value="0.1"/>
-    <!-- <inertia ixx="0.00095" iyy="0.000922" izz="4.7e-05" ixy="-0.0" iyz="-0.0" ixz="-0.0"/> -->
-    <inertia ixx="0.0" iyy="0.0" izz="0.0" ixy="0.0" iyz="0.0" ixz="0.0"/>
+    <inertia ixx="0.00095" iyy="0.000922" izz="4.7e-05" ixy="-0.0" iyz="-0.0" ixz="-0.0"/>
+    <!-- <inertia ixx="0.0" iyy="0.0" izz="0.0" ixy="0.0" iyz="0.0" ixz="0.0"/> -->
   </inertial>
   <visual>
@@ -301,9 +301,9 @@
   <limit upper="1.570796" lower="-1.570796" effort="100" velocity="100"/>
 </joint> -->
-<!-- <joint name="virtual_joint" type="fixed">
+<joint name="virtual_joint" type="fixed">
   <origin xyz="0.0 0.0 0.3" rpy="0.0 0.0 0.0"/>
   <parent link="world"/>
   <child link="base_link"/>
-</joint> -->
+</joint>
 <link name="leg_rb_tip">
 <visual>
