Commit message: added frames of odometry

File: quadruped_description/urdf/bot_urdf_hii.xacro (robot description, xacro)
@@ -1,5 +1,5 @@
 <?xml version="1.0" ?>
 <robot name="FusionComponent" xmlns:xacro="http://www.ros.org/wiki/xacro">
-<xacro:arg name="is_sim" default="true"/>
+<xacro:arg name="is_sim" default="false"/>
 <xacro:include filename="$(find quadruped_description)/urdf/materials.xacro" />
 <!-- <xacro:include filename="$(find quadruped_description)/urdf/bot_urdf_hii.trans" /> -->
@@ -15,5 +15,6 @@
   </inertial>
 </xacro:macro>
-<link name="world"></link>
+<!-- <link name="world"></link> -->
+<!-- <link name="base_footprint"></link> -->
 <link name="base_link">
   <!-- <inertial>
@@ -301,9 +302,9 @@
   <limit upper="1.570796" lower="-1.570796" effort="100" velocity="100"/>
 </joint> -->
-<joint name="virtual_joint" type="fixed">
+<!-- <joint name="virtual_joint" type="fixed">
   <origin xyz="0.0 0.0 0.3" rpy="0.0 0.0 0.0"/>
   <parent link="world"/>
   <child link="base_link"/>
-</joint>
+</joint> -->
 <link name="leg_rb_tip">
 <visual>
@@ -402,4 +403,9 @@
         </collision>
 </link>
+<!-- <joint name="footprint_joint" type="fixed">
+  <origin xyz="0.0 0.0 0.0" rpy="0 0 0"/>
+  <parent link="base_link"/>
+  <child link="base_footprint"/>
+</joint> -->
 <joint name="lb1_base" type="revolute">
   <origin xyz="0.159093 -0.13841 0.359825" rpy="0 0 0"/>

Commit message: changed urdf for stability

File: quadruped_description/urdf/bot_urdf_hii.xacro (robot description, xacro)
@@ -19,10 +19,11 @@
 <!-- <link name="base_footprint"></link> -->
 <link name="base_link">
-  <!-- <inertial>
-    <origin xyz="0.01 0.0 0.3459" rpy="0 0 0"/>
-    <mass value="2.5"/>
-    <inertia ixx="0.02245" iyy="0.02245" izz="0.02245" ixy="0.0" iyz="0.0" ixz="0.0"/>
-  </inertial> -->
-  <xacro:box_inertia m="1.0" l="0.10" w="0.244" h="0.27" xyz="0.01 0.0 0.3459" rpy="0 0 0" />
+<inertial>
+  <origin xyz="0 0 0" rpy="0 0 0"/>
+  <mass value="5.0"/>
+  <inertia ixx="0.02083" iyy="0.04167" izz="0.05417"
+           ixy="0.0" iyz="0.0" ixz="0.0"/>
+</inertial>
+  <!-- <xacro:box_inertia m="2.0" l="0.10" w="0.244" h="0.27" xyz="0.0 0.0 0.0" rpy="0 0 0" /> -->
   <visual>
     <origin xyz="0 0 0" rpy="0 0 0"/>
@@ -41,8 +42,8 @@
 <link name="lb1">
   <inertial>
-    <origin xyz="-0.025499639213758474 -0.03608650849380332 0.008837273060876838" rpy="0 0 0"/>
-    <mass value="0.01"/>
-    <inertia ixx="1.9e-05" iyy="1.9e-05" izz="1.9e-05" ixy="0.0" iyz="0.0" ixz="0.0"/>
-    <!-- <inertia ixx="0.0" iyy="0.0" izz="0.0" ixy="0.0" iyz="0.0" ixz="0.0"/> -->
+    <origin xyz="-0.0255 -0.0361 0.0088" rpy="0 0 0"/>
+    <mass     value="0.1"/>
+    <inertia  ixx="3.3e-05" iyy="3.3e-05" izz="6.7e-06"
+              ixy="0.0"     iyz="0.0"     ixz="0.0"/>
   </inertial>
   <visual>
@@ -61,9 +62,9 @@
 </link>
 <link name="lf1">
-  <inertial>
-    <origin xyz="-0.025499639213758293 -0.03608650849380346 0.008837273060876838" rpy="0 0 0"/>
-    <mass value="0.01"/>
-    <inertia ixx="1.9e-05" iyy="1.9e-05" izz="1.9e-05" ixy="0.0" iyz="0.0" ixz="0.0"/>
-    <!-- <inertia ixx="0.0" iyy="0.0" izz="0.0" ixy="0.0" iyz="0.0" ixz="0.0"/> -->
+ <inertial>
+    <origin xyz="-0.0255  0.0361 0.0088" rpy="0 0 0"/> <!-- mirrored Y -->
+    <mass     value="0.1"/>
+    <inertia  ixx="3.3e-05" iyy="3.3e-05" izz="6.7e-06"
+              ixy="0.0"     iyz="0.0"     ixz="0.0"/>
   </inertial>
   <visual>
@@ -82,9 +83,9 @@
 </link>
 <link name="rb1">
-  <inertial>
-    <origin xyz="-0.02549946018937349 0.03608721798818135 0.008837273060868067" rpy="0 0 0"/>
-    <mass value="0.01"/>
-    <inertia ixx="1.9e-05" iyy="1.9e-05" izz="1.9e-05" ixy="0.0" iyz="0.0" ixz="0.0"/>
-    <!-- <inertia ixx="0.0" iyy="0.0" izz="0.0" ixy="0.0" iyz="0.0" ixz="0.0"/> -->
+   <inertial>
+    <origin xyz="-0.0255  0.0361 0.0088" rpy="0 0 0"/> <!-- mirrored Y -->
+    <mass     value="0.1"/>
+    <inertia  ixx="3.3e-05" iyy="3.3e-05" izz="6.7e-06"
+              ixy="0.0"     iyz="0.0"     ixz="0.0"/>
   </inertial>
   <visual>
@@ -104,8 +105,8 @@
 <link name="rf1">
   <inertial>
-    <origin xyz="-0.025499460189373144 0.0360872179881816 0.008837273060868123" rpy="0 0 0"/>
-    <mass value="0.01"/>
-    <inertia ixx="1.9e-05" iyy="1.9e-05" izz="1.9e-05" ixy="0.0" iyz="0.0" ixz="0.0"/>
-    <!-- <inertia ixx="0.0" iyy="0.0" izz="0.0" ixy="0.0" iyz="0.0" ixz="0.0"/> -->
+    <origin xyz="-0.0255  0.0361 0.0088" rpy="0 0 0"/> <!-- mirrored Y -->
+    <mass     value="0.1"/>
+    <inertia  ixx="3.3e-05" iyy="3.3e-05" izz="6.7e-06"
+              ixy="0.0"     iyz="0.0"     ixz="0.0"/>
   </inertial>
   <visual>
@@ -124,9 +125,9 @@
 </link>
 <link name="lb2">
-  <inertial>
-    <origin xyz="4.4053550116163187e-07 -0.024997352134525086 -0.058" rpy="0 0 0"/>
-    <mass value="0.1"/>
-    <inertia ixx="0.00095" iyy="0.000922" izz="4.7e-05" ixy="-0.0" iyz="-0.0" ixz="-0.0"/>
-    <!-- <inertia ixx="0.0" iyy="0.0" izz="0.0" ixy="0.0" iyz="0.0" ixz="0.0"/> -->
+   <inertial>
+    <origin xyz="0.0 -0.0250 -0.058" rpy="0 0 0"/>
+    <mass     value="0.1"/>
+    <inertia  ixx="9.5e-04" iyy="9.22e-04" izz="4.7e-05"
+              ixy="0.0"     iyz="0.0"      ixz="0.0"/>
   </inertial>
   <visual>
@@ -145,9 +146,9 @@
 </link>
 <link name="lf2">
-  <inertial>
-    <origin xyz="4.4053550139755426e-07 -0.02499735213452492 -0.058" rpy="0 0 0"/>
-    <mass value="0.1"/>
-    <inertia ixx="0.00095" iyy="0.000922" izz="4.7e-05" ixy="-0.0" iyz="-0.0" ixz="-0.0"/>
-    <!-- <inertia ixx="0.0" iyy="0.0" izz="0.0" ixy="0.0" iyz="0.0" ixz="0.0"/> -->
+ <inertial>
+    <origin xyz="0.0 -0.0250 -0.058" rpy="0 0 0"/>
+    <mass     value="0.1"/>
+    <inertia  ixx="9.5e-04" iyy="9.22e-04" izz="4.7e-05"
+              ixy="0.0"     iyz="0.0"      ixz="0.0"/>
   </inertial>
   <visual>
@@ -167,8 +168,8 @@
 <link name="rb2">
   <inertial>
-    <origin xyz="4.405355014946988e-07 0.025002647865472988 -0.058" rpy="0 0 0"/>
-    <mass value="0.1"/>
-    <inertia ixx="0.00095" iyy="0.000922" izz="4.7e-05" ixy="-0.0" iyz="-0.0" ixz="-0.0"/>
-    <!-- <inertia ixx="0.0" iyy="0.0" izz="0.0" ixy="0.0" iyz="0.0" ixz="0.0"/> -->
+    <origin xyz="0.0  0.0250 -0.058" rpy="0 0 0"/>  <!-- mirrored Y -->
+    <mass     value="0.1"/>
+    <inertia  ixx="9.5e-04" iyy="9.22e-04" izz="4.7e-05"
+              ixy="0.0"     iyz="0.0"      ixz="0.0"/>
   </inertial>
   <visual>
@@ -187,11 +188,11 @@
 </link>
 <link name="rf2">
-  <!-- <inertial>
-    <origin xyz="4.4053550166123223e-07 0.025002647865473154 -0.058" rpy="0 0 0"/>
-    <mass value="0.1"/> -->
-    <!-- <inertia ixx="0.00095" iyy="0.000922" izz="4.7e-05" ixy="-0.0" iyz="-0.0" ixz="-0.0"/> -->
-    <!-- <inertia ixx="0.0" iyy="0.0" izz="0.0" ixy="0.0" iyz="0.0" ixz="0.0"/>
-  </inertial> -->
-  <xacro:box_inertia m="0.1" l="0.10" w="0.03" h="0.03" xyz="1.905177073602271e-07 -0.02550497548458827 -0.06999107230321813" rpy="0 0 0" />
+  <inertial>
+    <origin xyz="0.0  0.0250 -0.058" rpy="0 0 0"/>  <!-- mirrored Y -->
+    <mass     value="0.1"/>
+    <inertia  ixx="9.5e-04" iyy="9.22e-04" izz="4.7e-05"
+              ixy="0.0"     iyz="0.0"      ixz="0.0"/>
+  </inertial>
+  <!-- <xacro:box_inertia m="0.1" l="0.10" w="0.03" h="0.03" xyz="1.905177073602271e-07 -0.02550497548458827 -0.06999107230321813" rpy="0 0 0" /> -->
   <visual>
     <origin xyz="0.111407 -0.16059 -0.359825" rpy="0 0 0"/>
@@ -209,11 +210,11 @@
 </link>
 <link name="lb3">
-  <!-- <inertial>
-    <origin xyz="1.905177073602271e-07 -0.02550497548458827 -0.06999107230321813" rpy="0 0 0"/>
-    <mass value="0.1"/>
-    <inertia ixx="6.5e-05" iyy="6.3e-05" izz="6e-06" ixy="-0.0" iyz="-0.0" ixz="0.0"/> -->
-    <!-- <inertia ixx="0.0" iyy="0.0" izz="0.0" ixy="0.0" iyz="0.0" ixz="0.0"/> -->
-  <!-- </inertial> -->
-  <xacro:box_inertia m="0.1" l="0.10" w="0.03" h="0.03" xyz="1.905177073602271e-07 -0.02550497548458827 -0.06999107230321813" rpy="0 0 0" />
+  <inertial>
+    <origin xyz="0.0 -0.0255 -0.070" rpy="0 0 0"/>
+    <mass     value="0.1"/>
+    <inertia  ixx="6.5e-05" iyy="6.3e-05" izz="6.0e-06"
+              ixy="0.0"     iyz="0.0"     ixz="0.0"/>
+  </inertial>
+  <!-- <xacro:box_inertia m="0.1" l="0.10" w="0.03" h="0.03" xyz="1.905177073602271e-07 -0.02550497548458827 -0.06999107230321813" rpy="0 0 0" /> -->
   <visual>
     <origin xyz="-0.133593 0.16741 -0.205825" rpy="0 0 0"/>
@@ -231,11 +232,11 @@
 </link>
 <link name="lf3">
-  <!-- <inertial>
-    <origin xyz="1.905177022532012e-07 -0.025504975484588632 -0.06999107230321808" rpy="0 0 0"/>
-    <mass value="0.1"/>
-    <inertia ixx="6.5e-05" iyy="6.3e-05" izz="6e-06" ixy="-0.0" iyz="-0.0" ixz="0.0"/> -->
-    <!-- <inertia ixx="0.0" iyy="0.0" izz="0.0" ixy="0.0" iyz="0.0" ixz="0.0"/> -->
-  <!-- </inertial> -->
-  <xacro:box_inertia m="0.1" l="0.10" w="0.03" h="0.03" xyz="1.905177022532012e-07 -0.025504975484588632 -0.06999107230321808" rpy="0 0 0" />
+  <inertial>
+    <origin xyz="0.0 -0.0255 -0.070" rpy="0 0 0"/>
+    <mass     value="0.1"/>
+    <inertia  ixx="6.5e-05" iyy="6.3e-05" izz="6.0e-06"
+              ixy="0.0"     iyz="0.0"     ixz="0.0"/>
+  </inertial>
+  <!-- <xacro:box_inertia m="0.1" l="0.10" w="0.03" h="0.03" xyz="1.905177022532012e-07 -0.025504975484588632 -0.06999107230321808" rpy="0 0 0" /> -->
   <visual>
     <origin xyz="0.111407 0.16741 -0.205825" rpy="0 0 0"/>
@@ -253,11 +254,11 @@
 </link>
 <link name="rb3">
-  <!-- <inertial>
-    <origin xyz="7.100791705461074e-07 0.02550568497895228 -0.06999107230322818" rpy="0 0 0"/>
-    <mass value="0.1"/>
-    <inertia ixx="6.5e-05" iyy="6.3e-05" izz="6e-06" ixy="-0.0" iyz="0.0" ixz="-0.0"/> -->
-    <!-- <inertia ixx="0.0" iyy="0.0" izz="0.0" ixy="0.0" iyz="0.0" ixz="0.0"/> -->
-  <!-- </inertial> -->
-  <xacro:box_inertia m="0.1" l="0.10" w="0.03" h="0.03" xyz="7.100791705461074e-07 0.02550568497895228 -0.06999107230322818" rpy="0 0 0" />
+ <inertial>
+    <origin xyz="0.0  0.0255 -0.070" rpy="0 0 0"/> <!-- mirrored Y -->
+    <mass     value="0.1"/>
+    <inertia  ixx="6.5e-05" iyy="6.3e-05" izz="6.0e-06"
+              ixy="0.0"     iyz="0.0"     ixz="0.0"/>
+  </inertial>
+  <!-- <xacro:box_inertia m="0.1" l="0.10" w="0.03" h="0.03" xyz="7.100791705461074e-07 0.02550568497895228 -0.06999107230322818" rpy="0 0 0" /> -->
   <visual>
     <origin xyz="-0.133593 -0.16059 -0.205825" rpy="0 0 0"/>
@@ -275,11 +276,11 @@
 </link>
 <link name="rf3">
-  <!-- <inertial>
-    <origin xyz="7.100791702685516e-07 0.025505684978952448 -0.06999107230322804" rpy="0 0 0"/>
-    <mass value="0.1"/>
-    <inertia ixx="6.5e-05" iyy="6.3e-05" izz="6e-06" ixy="-0.0" iyz="0.0" ixz="-0.0"/> -->
-    <!-- <inertia ixx="0.0" iyy="0.0" izz="0.0" ixy="0.0" iyz="0.0" ixz="0.0"/> -->
-  <!-- </inertial> -->
-  <xacro:box_inertia m="0.1" l="0.10" w="0.03" h="0.03" xyz="7.100791702685516e-07 0.025505684978952448 -0.06999107230322804" rpy="0 0 0" />
+  <inertial>
+    <origin xyz="0.0  0.0255 -0.070" rpy="0 0 0"/> <!-- mirrored Y -->
+    <mass     value="0.1"/>
+    <inertia  ixx="6.5e-05" iyy="6.3e-05" izz="6.0e-06"
+              ixy="0.0"     iyz="0.0"     ixz="0.0"/>
+  </inertial>
+  <!-- <xacro:box_inertia m="0.1" l="0.10" w="0.03" h="0.03" xyz="7.100791702685516e-07 0.025505684978952448 -0.06999107230322804" rpy="0 0 0" /> -->
   <visual>
     <origin xyz="0.111407 -0.16059 -0.205825" rpy="0 0 0"/>
@@ -309,4 +310,12 @@
 </joint> -->
 <link name="leg_rb_tip">
+<inertial>
+    <origin xyz="0 0 0" rpy="0 0 0"/>
+    <mass value="0.01"/> <!-- 10 grams -->
+    <!-- Inertia of solid sphere: I = (2/5) * m * r^2 -->
+    <inertia
+      ixx="5.12e-08" iyy="5.12e-08" izz="5.12e-08"
+      ixy="0.0" iyz="0.0" ixz="0.0"/>
+  </inertial>
 <visual>
             <origin rpy="0 0 0" xyz="0 0 0"/>
@@ -333,4 +342,12 @@
 </link>
 <link name="leg_rf_tip">
+<inertial>
+    <origin xyz="0 0 0" rpy="0 0 0"/>
+    <mass value="0.01"/> <!-- 10 grams -->
+    <!-- Inertia of solid sphere: I = (2/5) * m * r^2 -->
+    <inertia
+      ixx="5.12e-08" iyy="5.12e-08" izz="5.12e-08"
+      ixy="0.0" iyz="0.0" ixz="0.0"/>
+  </inertial>
 <visual>
             <origin rpy="0 0 0" xyz="0 0 0"/>
@@ -357,4 +374,12 @@
 </link>
 <link name="leg_lb_tip">
+<inertial>
+    <origin xyz="0 0 0" rpy="0 0 0"/>
+    <mass value="0.01"/> <!-- 10 grams -->
+    <!-- Inertia of solid sphere: I = (2/5) * m * r^2 -->
+    <inertia
+      ixx="5.12e-08" iyy="5.12e-08" izz="5.12e-08"
+      ixy="0.0" iyz="0.0" ixz="0.0"/>
+  </inertial>
 <visual>
             <origin rpy="0 0 0" xyz="0 0 0"/>
@@ -381,4 +406,12 @@
 </link>
 <link name="leg_lf_tip">
+<inertial>
+    <origin xyz="0 0 0" rpy="0 0 0"/>
+    <mass value="0.01"/> <!-- 10 grams -->
+    <!-- Inertia of solid sphere: I = (2/5) * m * r^2 -->
+    <inertia
+      ixx="5.12e-08" iyy="5.12e-08" izz="5.12e-08"
+      ixy="0.0" iyz="0.0" ixz="0.0"/>
+  </inertial>
 <visual>
             <origin rpy="0 0 0" xyz="0 0 0"/>

Commit message: 2kg base mass, walking fine but controllers spawning is till now also not robust

File: quadruped_description/urdf/bot_urdf_hii.xacro (robot description, xacro)
@@ -21,6 +21,6 @@
 <inertial>
   <origin xyz="0 0 0" rpy="0 0 0"/>
-  <mass value="5.0"/>
-  <inertia ixx="0.02083" iyy="0.04167" izz="0.05417"
+  <mass value="2.0"/>
+  <inertia ixx="0.02303" iyy="0.02023" izz="0.03840"
            ixy="0.0" iyz="0.0" ixz="0.0"/>
 </inertial>

Commit message: 2kg base, increase mass of 3rd link of legs to 200g

File: quadruped_description/urdf/bot_urdf_hii.xacro (robot description, xacro)
@@ -211,9 +211,9 @@
 <link name="lb3">
   <inertial>
-    <origin xyz="0.0 -0.0255 -0.070" rpy="0 0 0"/>
-    <mass     value="0.1"/>
-    <inertia  ixx="6.5e-05" iyy="6.3e-05" izz="6.0e-06"
-              ixy="0.0"     iyz="0.0"     ixz="0.0"/>
-  </inertial>
+  <origin xyz="0.0 -0.0255 -0.070" rpy="0 0 0"/>
+  <mass value="0.2"/>
+  <inertia ixx="0.00013" iyy="0.000126" izz="0.000012"
+           ixy="0.0" iyz="0.0" ixz="0.0"/>
+</inertial>
   <!-- <xacro:box_inertia m="0.1" l="0.10" w="0.03" h="0.03" xyz="1.905177073602271e-07 -0.02550497548458827 -0.06999107230321813" rpy="0 0 0" /> -->
   <visual>
@@ -233,9 +233,9 @@
 <link name="lf3">
   <inertial>
-    <origin xyz="0.0 -0.0255 -0.070" rpy="0 0 0"/>
-    <mass     value="0.1"/>
-    <inertia  ixx="6.5e-05" iyy="6.3e-05" izz="6.0e-06"
-              ixy="0.0"     iyz="0.0"     ixz="0.0"/>
-  </inertial>
+  <origin xyz="0.0 -0.0255 -0.070" rpy="0 0 0"/>
+  <mass value="0.2"/>
+  <inertia ixx="0.00013" iyy="0.000126" izz="0.000012"
+           ixy="0.0" iyz="0.0" ixz="0.0"/>
+</inertial>
   <!-- <xacro:box_inertia m="0.1" l="0.10" w="0.03" h="0.03" xyz="1.905177022532012e-07 -0.025504975484588632 -0.06999107230321808" rpy="0 0 0" /> -->
   <visual>
@@ -254,10 +254,10 @@
 </link>
 <link name="rb3">
- <inertial>
-    <origin xyz="0.0  0.0255 -0.070" rpy="0 0 0"/> <!-- mirrored Y -->
-    <mass     value="0.1"/>
-    <inertia  ixx="6.5e-05" iyy="6.3e-05" izz="6.0e-06"
-              ixy="0.0"     iyz="0.0"     ixz="0.0"/>
-  </inertial>
+<inertial>
+  <origin xyz="0.0 -0.0255 -0.070" rpy="0 0 0"/>
+  <mass value="0.2"/>
+  <inertia ixx="0.00013" iyy="0.000126" izz="0.000012"
+           ixy="0.0" iyz="0.0" ixz="0.0"/>
+</inertial>
   <!-- <xacro:box_inertia m="0.1" l="0.10" w="0.03" h="0.03" xyz="7.100791705461074e-07 0.02550568497895228 -0.06999107230322818" rpy="0 0 0" /> -->
   <visual>
@@ -277,9 +277,9 @@
 <link name="rf3">
   <inertial>
-    <origin xyz="0.0  0.0255 -0.070" rpy="0 0 0"/> <!-- mirrored Y -->
-    <mass     value="0.1"/>
-    <inertia  ixx="6.5e-05" iyy="6.3e-05" izz="6.0e-06"
-              ixy="0.0"     iyz="0.0"     ixz="0.0"/>
-  </inertial>
+  <origin xyz="0.0 -0.0255 -0.070" rpy="0 0 0"/>
+  <mass value="0.2"/>
+  <inertia ixx="0.00013" iyy="0.000126" izz="0.000012"
+           ixy="0.0" iyz="0.0" ixz="0.0"/>
+</inertial>
   <!-- <xacro:box_inertia m="0.1" l="0.10" w="0.03" h="0.03" xyz="7.100791702685516e-07 0.025505684978952448 -0.06999107230322804" rpy="0 0 0" /> -->
   <visual>
